Commit message: update

File: urdf/my_robot.xacro (robot description, xacro)
@@ -1,6 +1,5 @@
 <?xml version='1.0'?>
-<!-- csosa_bot -->
 <robot name="udacity_bot" xmlns:xacro="http://www.ros.org/wiki/xacro">
-  <xacro:include filename="$(find udacity_bot)/urdf/my_bot.gazebo"/>
+  <xacro:include filename="$(find udacity_bot)/urdf/my_robot.gazebo"/>
   <link name="robot_footprint"></link>
   <joint name="robot_footprint_joint" type="fixed">
@@ -13,5 +12,5 @@
     <pose>0 0 0.1 0 0 0</pose>
     <inertial>
-      <mass value="10.0"/>
+      <mass value="20.0"/>
       <origin xyz="0.0 0 0" rpy=" 0 0 0"/>
       <inertia
@@ -32,6 +31,6 @@
         <cylinder radius="0.2" length="0.1"/>
       </geometry>
-      <material name="black">
-        <color rgba="0 0 0 1"/>
+      <material name="white">
+        <color rgba="1 1 1 1"/>
       </material>
     </visual>
@@ -81,5 +80,5 @@
     </visual>
   </link>
-  <!-- Left Wheel Link -->
+   <!-- Left Wheel Link -->
   <link name="left_wheel">
     <inertial>
@@ -94,14 +93,14 @@
     <visual>
       <geometry>
-        <cylinder length="0.05" radius="0.1"/>
-      </geometry>
-      <origin xyz="0 0 0" rpy="0 1.5707 1.5707"/>
-      <material name="white">
-        <color rgba="1 1 1 1"/>
-      </material>
-    </visual>
-    <collision>
-      <geometry>
-        <cylinder length="0.05" radius="0.1"/>
+        <cylinder length="0.1" radius="0.05"/>
+      </geometry>
+      <origin xyz="0 0 0" rpy="0 1.5707 1.5707"/>
+      <material name="black">
+        <color rgba="0 0 0 1"/>
+      </material>
+    </visual>
+    <collision>
+      <geometry>
+        <cylinder length="0.1" radius="0.05"/>
       </geometry>
       <origin xyz="0 0 0" rpy="0 1.5707 1.5707"/>
@@ -121,14 +120,14 @@
     <visual>
       <geometry>
-        <cylinder length="0.05" radius="0.1"/>
-      </geometry>
-      <origin xyz="0 0 0" rpy="0 1.5707 1.5707"/>
-      <material name="white">
-        <color rgba="1 1 1 1"/>
-      </material>
-    </visual>
-    <collision>
-      <geometry>
-        <cylinder length="0.05" radius="0.1"/>
+        <cylinder length="0.05" radius="0.05"/>
+      </geometry>
+      <origin xyz="0 0 0" rpy="0 1.5707 1.5707"/>
+      <material name="black">
+        <color rgba="0 0 0 1"/>
+      </material>
+    </visual>
+    <collision>
+      <geometry>
+        <cylinder length="0.05" radius="0.05"/>
       </geometry>
       <origin xyz="0 0 0" rpy="0 1.5707 1.5707"/>
@@ -188,26 +187,26 @@
   <!-- Joints -->
   <joint type="continuous" name="left_wheel_hinge">
-    <origin xyz="0 0.25 0" rpy="0 0 0"/>
+    <origin xyz="0 0.1 -0.05" rpy="0 0 0"/>
     <child link="left_wheel"/>
     <parent link="chassis"/>
-    <axis xyz="0 1 0" rpy="0 0 0"/>
+    <axis xyz="0 0.05 -0.05" rpy="0 0 0"/>
     <limit effort="10000" velocity="1000"/>
     <joint_properties damping="1.0" friction="1.0"/>
   </joint>
   <joint type="continuous" name="right_wheel_hinge">
-    <origin xyz="0 -0.25 0" rpy="0 0 0"/>
+    <origin xyz="0 -0.1 -0.05" rpy="0 0 0"/>
     <child link="right_wheel"/>
     <parent link="chassis"/>
-    <axis xyz="0 1 0" rpy="0 0 0"/>
+    <axis xyz="0 -0.05 -0.05" rpy="0 0 0"/>
     <limit effort="10000" velocity="1000"/>
     <joint_properties damping="1.0" friction="1.0"/>
   </joint>
   <joint type="fixed" name="camera_joint">
-    <origin xyz="0.25 0 0" rpy="0 0 0"/>
+    <origin xyz="0.2 0 0" rpy="0 0 0"/>
     <child link="camera"/>
     <parent link="chassis"/>
   </joint>
   <joint type="fixed" name="hokuyo_joint">
-    <origin xyz="0.0 0 0.1" rpy="0 0 0"/>
+    <origin xyz="0.05 0 0.05" rpy="0 0 0"/>
     <child link="hokuyo"/>
     <parent link="chassis"/>

Commit message: update

File: urdf/my_robot.xacro (robot description, xacro)
@@ -93,5 +93,5 @@
     <visual>
       <geometry>
-        <cylinder length="0.1" radius="0.05"/>
+        <cylinder length="0.05" radius="0.05"/>
       </geometry>
       <origin xyz="0 0 0" rpy="0 1.5707 1.5707"/>
@@ -102,5 +102,5 @@
     <collision>
       <geometry>
-        <cylinder length="0.1" radius="0.05"/>
+        <cylinder length="0.05" radius="0.05"/>
       </geometry>
       <origin xyz="0 0 0" rpy="0 1.5707 1.5707"/>
@@ -187,16 +187,16 @@
   <!-- Joints -->
   <joint type="continuous" name="left_wheel_hinge">
-    <origin xyz="0 0.1 -0.05" rpy="0 0 0"/>
+    <origin xyz="0 0.15 -0.05" rpy="0 0 0"/>
     <child link="left_wheel"/>
     <parent link="chassis"/>
-    <axis xyz="0 0.05 -0.05" rpy="0 0 0"/>
+    <axis xyz="0 1 0" rpy="0 0 0"/>
     <limit effort="10000" velocity="1000"/>
     <joint_properties damping="1.0" friction="1.0"/>
   </joint>
   <joint type="continuous" name="right_wheel_hinge">
-    <origin xyz="0 -0.1 -0.05" rpy="0 0 0"/>
+    <origin xyz="0 -0.15 -0.05" rpy="0 0 0"/>
     <child link="right_wheel"/>
     <parent link="chassis"/>
-    <axis xyz="0 -0.05 -0.05" rpy="0 0 0"/>
+    <axis xyz="0 1 0" rpy="0 0 0"/>
     <limit effort="10000" velocity="1000"/>
     <joint_properties damping="1.0" friction="1.0"/>
